Commit message: add color to person model

File: src/body_description/urdf/body.xacro (robot description, xacro)
@@ -15,5 +15,4 @@
       <mesh filename="package://body_description/meshes/base_link.stl" scale="0.001 0.001 0.001"/>
     </geometry>
-    <material name="steel_satin"/>
   </visual>
   <collision>
@@ -24,3 +23,6 @@
   </collision>
 </link>
+<gazebo reference="base_link">
+  <material>Gazebo/Blue</material>
+</gazebo>
 </robot>
